File: pcb/motor.brd (EAGLE design)
At the start: 15.5 x 27.9 mm, 8 parts, among them Q1 BC847, X1 X1

Commit message: Added an extra pad for the control signal on motor board.
Parts:
- M1: value B/C11L -> ada1201
- renumbered SG1 to M1
Changed lines of the file:
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@@
 <elements>
 <element name="Q1" library="transistor-npn" package="SOT23" value="BC847" x="11.43" y="7.62" smashed="yes" rot="R270"/>
-<element name="SG1" library="buzzer" package="B/C11L" value="B/C11L" x="7.62" y="19.05" smashed="yes">
+<element name="M1" library="buzzer" package="B/C11L" value="ada1201" x="7.62" y="19.05" smashed="yes">
 <attribute name="OC_NEWARK" value="unknown" x="7.62" y="19.05" size="1.778" layer="27" display="off"/>
 <attribute name="MPN" value="" x="7.62" y="19.05" size="1.778" layer="27" display="off"/>
@@
 <contactref element="D1" pad="A"/>
 <contactref element="C1" pad="2"/>
-<contactref element="SG1" pad="2"/>
+<contactref element="M1" pad="2"/>
 <wire x1="11.43" y1="11.43" x2="8.89" y2="11.43" width="0.762" layer="1"/>
 <wire x1="8.89" y1="11.43" x2="8.47" y2="11.43" width="0.762" layer="1"/>
@@
 <contactref element="D1" pad="C"/>
 <contactref element="C1" pad="1"/>
-<contactref element="SG1" pad="1"/>
+<contactref element="M1" pad="1"/>
 <contactref element="R2" pad="2"/>
 <wire x1="3.81" y1="11.43" x2="6.77" y2="11.43" width="0.762" layer="1"/>
